File: carte_RPI5_KiCad/carte_rpi5_kicad.kicad_sch (KiCad schematic)
At the start: 0 parts

Commit message: Placement composants
Parts:
- added PS1: OKL-T_6-W12N-C, OKLT6W12NC, symbol Librairie_symbole:OKL-T_6-W12N-C
- added U1: CM5108032, CM5108032:MODULE_CM5108032, symbol Librairie_symbole:CM5108032
- added U2: BNO055, BNO055:LGA28R50P4X10_380X520X100, symbol Librairie_symbole:BNO055
- added U3: L293D, L293D:DIP880W50P254L2000H510Q16, symbol Librairie_symbole:L293D
- added U4: LPS22HB, LPS22HB:LGA10R50P2X3_200X200X80, symbol Librairie_symbole:LPS22HB
- added U5: PCA9685PW_118, PCA9685PW_118:SOP65P640X110-28N, symbol Librairie_symbole:PCA9685PW_118
Connections:
- new net: U1.SH1 (MOUNTING_PADS), U1.SH2 (MOUNTING_PADS), U1.SH3 (MOUNTING_PADS), U1.SH4 (MOUNTING_PADS)
- new net +5V(INPUT): U1.77 (+5V(INPUT)), U1.79 (+5V(INPUT)), U1.81 (+5V(INPUT)), U1.83 (+5V(INPUT)), U1.85 (+5V(INPUT)), U1.87 (+5V(INPUT))
- new net CM5_1.8V(OUTPUT): U1.88 (CM5_1.8V(OUTPUT)), U1.90 (CM5_1.8V(OUTPUT))
- new net CM5_3.3V(OUTPUT): U1.84 (CM5_3.3V(OUTPUT)), U1.86 (CM5_3.3V(OUTPUT))
- new net GND: U1.1 (GND), U1.107 (GND), U1.108 (GND), U1.113 (GND), U1.114 (GND), U1.119 (GND), U1.120 (GND), U1.125 (GND), U1.126 (GND), U1.13 (GND), U1.131 (GND), U1.132 (GND), U1.137 (GND), U1.138 (GND), U1.14 (GND), U1.144 (GND), U1.150 (GND), U1.155 (GND), U1.156 (GND), U1.161 (GND), U1.162 (GND), U1.167 (GND), U1.168 (GND), U1.173 (GND), U1.174 (GND), U1.179 (GND), U1.180 (GND), U1.185 (GND), U1.186 (GND), U1.191 (GND), U1.192 (GND), U1.197 (GND), U1.198 (GND), U1.2 (GND), U1.22 (GND), U1.23 (GND), U1.32 (GND), U1.33 (GND), U1.42 (GND), U1.43 (GND), U1.52 (GND), U1.53 (GND), U1.59 (GND), U1.60 (GND), U1.65 (GND), U1.66 (GND), U1.7 (GND), U1.71 (GND), U1.74 (GND), U1.8 (GND), U1.98 (GND), U3.12 (GND), U3.13 (GND), U3.4 (GND), U3.5 (GND), U4.8 (GND), U4.9 (GND)

Commit message: Début du schéma Kicad
Parts:
- removed PS1: OKL-T_6-W12N-C, OKLT6W12NC, symbol Librairie_symbole:OKL-T_6-W12N-C
- added C1: 1uF, symbol Device:C
- added C2: 120nF, symbol Device:C
- added D1: LED, LED_SMD:LED_0805_2012Metric, symbol Device:LED
- added F1: Fuse, Fuse:Fuse_0402_1005Metric, symbol Device:Fuse
- added J1: Vin Batterie, TerminalBlock:TerminalBlock_MaiXu_MX126-5.0-02P_1x02_P5.00mm, symbol Connector:Screw_Terminal_01x02
- added R1: 220, Resistor_SMD:R_0805_2012Metric, symbol Device:R
- added R2: 1340, Resistor_SMD:R_0805_2012Metric, symbol Device:R
- added R_Pull (x2): R, symbol Device:R
- added Régulateur_de_tension: OKL-T_6-W12N-C, Library:OKLT6W12NC, symbol OKL-T_6-W12N-C:OKL-T_6-W12N-C
- added SW1: SW_SPDT, Button_Switch_THT:SW_DIP_SPSTx01_Slide_6.7x4.1mm_W7.62mm_P2.54mm_LowProfile, symbol Switch:SW_SPDT
- renumbered U4 to Capteur_de_Pression, U2 to Centrale_Inertielle, U5 to Contrôleur_PWM, U3 to Pont_en_H, U1 to Raspberry5
Connections:
- net +5V(INPUT): now also Régulateur_de_tension.4 (VOUT), Régulateur_de_tension.5 (SENSE)
- net CM5_3.3V(OUTPUT): now also Centrale_Inertielle.28 (VDDIO), Centrale_Inertielle.3 (VDD), Contrôleur_PWM.28 (VDD), C2.2, R_Pull.1
- net GND: now also Centrale_Inertielle.2 (GND), Contrôleur_PWM.1 (A0), Contrôleur_PWM.14 (VSS), Contrôleur_PWM.2 (A1), Contrôleur_PWM.24 (A5), Contrôleur_PWM.25 (EXTCLK), Contrôleur_PWM.3 (A2), Contrôleur_PWM.4 (A3), Contrôleur_PWM.5 (A4), D1.1 (K), J1.1 (Pin_1), R2.2, Régulateur_de_tension.3 (GROUND_1), Régulateur_de_tension.7 (GROUND_2), SW1.2 (B)
- net I2C_ADDR_SEL: now reaches Centrale_Inertielle.17 (COM3)
- net SCL: now reaches Centrale_Inertielle.19 (COM1)
- net SCL: now also Contrôleur_PWM.26 (SCL), R_Pull.2
- net SDA: now reaches Centrale_Inertielle.20 (COM0)
- net SDA: now also Contrôleur_PWM.27 (SDA), R_Pull.1, R_Pull.2
- net at Centrale_Inertielle.25 (GNDIO): now also C2.1
- net at Centrale_Inertielle.9 (CAP): now also C1.2
- net PWM4: now reaches Contrôleur_PWM.10 (LED4)
- net PWM5: now reaches Contrôleur_PWM.11 (LED5)
- net PWM6: now reaches Contrôleur_PWM.12 (LED6)
- net PWM7: now reaches Contrôleur_PWM.13 (LED7)
- net PWM0: now reaches Contrôleur_PWM.6 (LED0)
- net PWM1: now reaches Contrôleur_PWM.7 (LED1)
- net PWM2: now reaches Contrôleur_PWM.8 (LED2)
- net PWM3: now reaches Contrôleur_PWM.9 (LED3)
- new net: D1.2 (A), R1.1
- new net: F1.1, J1.2 (Pin_2)
- new net: R2.1, Régulateur_de_tension.6 (TRIM)
- new net: R1.2, Régulateur_de_tension.10 (POWER_GOOD_OUT)
- new net: Régulateur_de_tension.1 (ON/OFF_CONTROL), SW1.1 (A)
- new net: F1.2, Régulateur_de_tension.2 (VIN)
Other:
- note added: "Contrôleur_PWM"
- note added: "Demander à Thomas résistance sur interrupteur"
- note added: "Demander à Thomas si l'empreinte est bonne Où trouver l'empreinte du site du fabricant"
- note added: "Peut-on le monter en surface?"
- note added: "Rajouter des pins pour le moteur ; demander à Thomas pour les empreintes des pins"
- note added: "Régulateur de Tension (7V -> 5V)"
- moved on the sheet: Capteur_de_Pression, Centrale_Inertielle, Contrôleur_PWM, Pont_en_H, Raspberry5A

Commit message: Modif kicad
Parts:
- added J1, J2, J3, J4, J5, J6, J7, J8: Conn_01x03, symbol Connector_Generic:Conn_01x03
- added R_Pull_Up: 1 k, symbol Device:R
Connections:
- net +5V(INPUT): now also J1.2 (Pin_2), J2.2 (Pin_2), J3.2 (Pin_2), J4.2 (Pin_2), J5.2 (Pin_2), J6.2 (Pin_2), J7.2 (Pin_2), J8.2 (Pin_2)
- net GND: now also J1.1 (Pin_1), J2.1 (Pin_1), J3.1 (Pin_1), J4.1 (Pin_1), J5.1 (Pin_1), J6.1 (Pin_1), J7.1 (Pin_1), J8.1 (Pin_1)
- net PWM0: now also J1.3 (Pin_3)
- net PWM1: now also J2.3 (Pin_3)
- net PWM2: now also J3.3 (Pin_3)
- net PWM3: now also J4.3 (Pin_3)
- net PWM4: now also J5.3 (Pin_3)
- net PWM5: now also J6.3 (Pin_3)
- net PWM6: now also J7.3 (Pin_3)
- net PWM7: now also J8.3 (Pin_3)
- net at Régulateur_de_tension.1 (ON/OFF_CONTROL), SW1.1 (A): now also R_Pull_Up.2
- net at F1.2, Régulateur_de_tension.2 (VIN): now also R_Pull_Up.1
Other:
- note added: "Connecteurs pour PWM"
- company: (none) -> ENS Paris-Saclay
- moved on the sheet: Capteur_de_Pression, Pont_en_H, Raspberry5A, SW1

Commit message: Kicad edit
Parts:
- added Conn_BNO, Conn_luna: Conn_01x04_Pin, symbol Connector:Conn_01x04_Pin
- added Conn_LPS22HB: Conn_01x08, symbol Connector_Generic:Conn_01x08
- added Conn_treuil_pince: Conn_01x05, symbol Connector_Generic:Conn_01x05
Connections:
- net CM5_3.3V(OUTPUT): now also Pont_en_H.1 (ENABLE1), Pont_en_H.16 (VSS), Pont_en_H.9 (ENABLE2), Conn_BNO.4 (Pin_4), Conn_LPS22HB.1 (Pin_1), Conn_luna.4 (Pin_4)
- net GND: now also Conn_BNO.1 (Pin_1), Conn_LPS22HB.3 (Pin_3), Conn_luna.1 (Pin_1), Conn_treuil_pince.1 (Pin_1)
- net SCL: now also Conn_BNO.2 (Pin_2), Conn_luna.2 (Pin_2)
- net SDA: now also Conn_BNO.3 (Pin_3), Conn_luna.3 (Pin_3)
- net PWM10: now reaches Pont_en_H.10 (INPUT3)
- net PWM10: now also Contrôleur_PWM.17 (LED10)
- net Mot_pince+: now reaches Pont_en_H.11 (OUTPUT3)
- net Mot_pince-: now reaches Pont_en_H.14 (OUTPUT4)
- net PWM11: now reaches Pont_en_H.15 (INPUT4)
- net PWM11: now also Contrôleur_PWM.18 (LED11)
- net PWM8: now reaches Pont_en_H.2 (INPUT1)
- net PWM8: now also Contrôleur_PWM.15 (LED8)
- net Mot_treuil+: now reaches Pont_en_H.3 (OUTPUT1)
- net Mot_treuil-: now reaches Pont_en_H.6 (OUTPUT2)
- net PWM9: now reaches Pont_en_H.7 (INPUT2)
- net PWM9: now also Contrôleur_PWM.16 (LED9)
- net V_bat: now reaches Pont_en_H.8 (VS)
Other:
- note added: "Centrale Inertielle non utilisée"
- note added: "Connecteur pour BNO055"
- note added: "Connecteur pour télémètre Luna"
- note added: "Connecteurs PWM pour les moteurs"
- note added: "Connecteurs pour le capteur de pression"
- note added: "Connecteurs pour moteurs treuil et pince"
- note added: "Pas beosin du I2C addr_sel car addresse déjà défini sur la centrale"
- note added: "Pont en H pour contrôler les moteurs treuil et pince"
- note removed: "Connecteurs pour PWM"
- company: ENS Paris-Saclay -> ENS Paris-Saclay - Anis SAMLALI, Matisse Morote--Humbert, Lucie Stagnavo, Lisa Wu
- title: (none) -> Schéma de la carte électronique principale - Projet COBRA 2025
- moved on the sheet: C1, C2, Capteur_de_Pression, Centrale_Inertielle, Contrôleur_PWM, R_Pull

Commit message: Empreinte OKL ok
Parts:
- removed Conn_treuil_pince: Conn_01x05, symbol Connector_Generic:Conn_01x05
- added Conn_pince, Conn_treuil: Conn_01x02, symbol Connector_Generic:Conn_01x02
- added R_SCL, R_SDA: 4,7k, symbol Device:R
- Régulateur_de_tension: footprint Library:OKLT6W12NC -> librairie_empreintes:OKLT6W12NC
Connections:
- net CM5_3.3V(OUTPUT): now also R_SCL.1, R_SDA.2
- net Mot_pince+: now also Conn_pince.2 (Pin_2)
- net Mot_pince-: now also Conn_pince.1 (Pin_1)
- net Mot_treuil+: now also Conn_treuil.2 (Pin_2)
- net Mot_treuil-: now also Conn_treuil.1 (Pin_1)
- net SCL: now also Conn_LPS22HB.4 (Pin_4), Raspberry5.57 (SD_CLK), R_SCL.2
- net SDA: now also Conn_LPS22HB.6 (Pin_6), Raspberry5.63 (SD_DAT0), R_SDA.1
Other:
- moved on the sheet: Conn_LPS22HB

Commit message: Add empeintes to carte_rpi5
Parts:
- removed Conn_pince, Conn_treuil: Conn_01x02, symbol Connector_Generic:Conn_01x02
- removed J1: Vin Batterie, TerminalBlock:TerminalBlock_MaiXu_MX126-5.0-02P_1x02_P5.00mm, symbol Connector:Screw_Terminal_01x02
- added Conn_Treuil_Pince1: Conn_01x04_Pin, Connector_PinSocket_2.54mm:PinSocket_1x04_P2.54mm_Vertical, symbol Connector:Conn_01x04_Pin
- added J0: Vin batterie, Connector_AMASS:AMASS_XT60-F_1x02_P7.20mm_Vertical, symbol Librairie_symbole:XT60-M
- Conn_BNO1: renamed from Conn_BNO; footprint (none) -> Connector_PinSocket_2.54mm:PinSocket_1x04_P2.54mm_Vertical
- Conn_LPS22HB1: renamed from Conn_LPS22HB; footprint (none) -> Connector_PinSocket_2.54mm:PinSocket_1x08_P2.54mm_Vertical
- Conn_luna1: renamed from Conn_luna; footprint (none) -> Connector_PinSocket_2.54mm:PinSocket_1x04_P2.54mm_Vertical
- Contrôleur_PWM1: renamed from Contrôleur_PWM; footprint PCA9685PW_118:SOP65P640X110-28N -> librairie_empreintes:SOP65P640X110-28N
- J1, J2, J3, J4, J5, J6, J7, J8: footprint (none) -> Connector_PinHeader_2.54mm:PinHeader_1x03_P2.54mm_Vertical
- Pont_en_H1: renamed from Pont_en_H; footprint L293D:DIP880W50P254L2000H510Q16 -> Package_DIP:CERDIP-16_W7.62mm_SideBrazed
- R_Pull_Up1: renamed from R_Pull_Up; footprint (none) -> Resistor_SMD:R_0805_2012Metric
- R_SCL1: renamed from R_SCL; footprint (none) -> Resistor_SMD:R_0805_2012Metric
- R_SDA1: renamed from R_SDA; footprint (none) -> Resistor_SMD:R_0805_2012Metric
- Raspberry5: footprint CM5108032:MODULE_CM5108032 -> Connector_PinSocket_2.54mm:PinSocket_2x20_P2.54mm_Vertical
- renumbered Capteur_de_Pression to Capteur_de_Pression1, Centrale_Inertielle to Centrale_Inertielle1, R_Pull to R_Pull1, R_Pull to R_Pull2, Régulateur_de_tension to Régulateur_de_tension1
Connections:
- net GND: now also J0.N (NEG)
- net Mot_pince+: now also Conn_Treuil_Pince1.1 (Pin_1)
- net Mot_pince-: now also Conn_Treuil_Pince1.2 (Pin_2)
- net Mot_treuil+: now also Conn_Treuil_Pince1.3 (Pin_3)
- net Mot_treuil-: now also Conn_Treuil_Pince1.4 (Pin_4)
- net at F1.1: now also J0.P (POS)

Commit message: pcb_V0.1
Parts:
- removed J0: Vin batterie, Connector_AMASS:AMASS_XT60-F_1x02_P7.20mm_Vertical, symbol Librairie_symbole:XT60-M
- added J9: XT60-M, XT60-M:AMASS_XT60-M, symbol Librairie_symbole:XT60-M
Connections:
- net GND: now also J9.1 (NEG)
- net at F1.1: now also J9.2 (POS)
Changed lines of the file:
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@@
 	(wire
 		(pts
-			(xy 29.21 43.18) (xy 29.21 41.91)
-		)
-		(stroke
-			(width 0)
-			(type default)
-		)
-	)
-	(wire
-		(pts
 			(xy 66.04 48.26) (xy 67.31 48.26)
 		)
@@
 	(wire
 		(pts
-			(xy 50.8 43.18) (xy 67.31 43.18)
+			(xy 29.21 43.18) (xy 38.1 43.18)
 		)
 		(stroke
@@
 	(wire
 		(pts
-			(xy 67.31 50.8) (xy 66.04 50.8)
+			(xy 50.8 43.18) (xy 67.31 43.18)
 		)
 		(stroke
@@
 	(wire
 		(pts
-			(xy 337.82 220.98) (xy 349.25 220.98)
+			(xy 67.31 50.8) (xy 66.04 50.8)
 		)
 		(stroke
@@
 	(wire
 		(pts
-			(xy 29.21 43.18) (xy 38.1 43.18)
+			(xy 337.82 220.98) (xy 349.25 220.98)
 		)
 		(stroke
@@
 	(wire
 		(pts
+			(xy 29.21 43.18) (xy 29.21 39.37)
+		)
+		(stroke
+			(width 0)
+			(type default)
+		)
+	)
+	(wire
+		(pts
 			(xy 242.57 48.26) (xy 247.65 48.26)
 		)
@@
 	(wire
 		(pts
-			(xy 26.67 41.91) (xy 26.67 44.45)
+			(xy 26.67 39.37) (xy 26.67 44.45)
 		)
 		(stroke
@@
 	)
 	(symbol
-		(lib_id "Librairie_symbole:XT60-M")
-		(at 26.67 36.83 270)
-		(mirror x)
-		(unit 1)
-		(exclude_from_sim no)
-		(in_bom yes)
-		(on_board yes)
-		(dnp no)
-		(property "Reference" "J0"
-			(at 21.59 30.226 90)
-			(effects
-				(font
-					(size 1.27 1.27)
-				)
-				(justify right)
-			)
-		)
-		(property "Value" "Vin batterie"
-			(at 26.67 27.686 90)
-			(effects
-				(font
-					(size 1.27 1.27)
-				)
-				(justify right)
-			)
-		)
-		(property "Footprint" "Connector_AMASS:AMASS_XT60-F_1x02_P7.20mm_Vertical"
-			(at 26.67 36.83 0)
-			(effects
-				(font
-					(size 1.27 1.27)
-				)
-				(justify bottom)
-				(hide yes)
-			)
-		)
-		(property "Datasheet" ""
-			(at 26.67 36.83 0)
-			(effects
-				(font
-					(size 1.27 1.27)
-				)
-				(hide yes)
-			)
-		)
-		(property "Description" ""
-			(at 26.67 36.83 0)
-			(effects
-				(font
-					(size 1.27 1.27)
-				)
-				(hide yes)
-			)
-		)
-		(property "MF" "AMASS"
-			(at 26.67 36.83 0)
-			(effects
-				(font
-					(size 1.27 1.27)
-				)
-				(justify bottom)
-				(hide yes)
-			)
-		)
-		(property "MAXIMUM_PACKAGE_HEIGHT" "16.00 mm"
-			(at 26.67 36.83 0)
-			(effects
-				(font
-					(size 1.27 1.27)
-				)
-				(justify bottom)
-				(hide yes)
-			)
-		)
-		(property "Package" "Package"
-			(at 26.67 36.83 0)
-			(effects
-				(font
-					(size 1.27 1.27)
-				)
-				(justify bottom)
-				(hide yes)
-			)
-		)
-		(property "Price" "None"
-			(at 26.67 36.83 0)
-			(effects
-				(font
-					(size 1.27 1.27)
-				)
-				(justify bottom)
-				(hide yes)
-			)
-		)
-		(property "Check_prices" "https://www.snapeda.com/parts/XT60-M/AMASS/view-part/?ref=eda"
-			(at 26.67 36.83 0)
-			(effects
-				(font
-					(size 1.27 1.27)
-				)
-				(justify bottom)
-				(hide yes)
-			)
-		)
-		(property "STANDARD" "IPC 7351B"
-			(at 26.67 36.83 0)
-			(effects
-				(font
-					(size 1.27 1.27)
-				)
-				(justify bottom)
-				(hide yes)
-			)
-		)
-		(property "PARTREV" "V1.2"
-			(at 26.67 36.83 0)
-			(effects
-				(font
-					(size 1.27 1.27)
-				)
-				(justify bottom)
-				(hide yes)
-			)
-		)
-		(property "SnapEDA_Link" "https://www.snapeda.com/parts/XT60-M/AMASS/view-part/?ref=snap"
-			(at 26.67 36.83 0)
-			(effects
-				(font
-					(size 1.27 1.27)
-				)
-				(justify bottom)
-				(hide yes)
-			)
-		)
-		(property "MP" "XT60-M"
-			(at 26.67 36.83 0)
-			(effects
-				(font
-					(size 1.27 1.27)
-				)
-				(justify bottom)
-				(hide yes)
-			)
-		)
-		(property "Description_1" "Plug; DC supply; XT60; male; PIN: 2; for cable; soldered; 30A; 500V"
-			(at 26.67 36.83 0)
-			(effects
-				(font
-					(size 1.27 1.27)
-				)
-				(justify bottom)
-				(hide yes)
-			)
-		)
-		(property "Availability" "In Stock"
-			(at 26.67 36.83 0)
-			(effects
-				(font
-					(size 1.27 1.27)
-				)
-				(justify bottom)
-				(hide yes)
-			)
-		)
-		(property "MANUFACTURER" "AMASS"
-			(at 26.67 36.83 0)
-			(effects
-				(font
-					(size 1.27 1.27)
-				)
-				(justify bottom)
-				(hide yes)
-			)
-		)
-		(pin "P"
-		)
-		(pin "N"
-		)
-		(instances
-			(project ""
-				(path "/1781f24e-6d21-4940-8f28-5db05927caba"
-					(reference "J0")
-					(unit 1)
-				)
-			)
-		)
-	)
-	(symbol
 		(lib_id "Device:R")
 		(at 332.74 220.98 90)
@@
 					(unit 1)
 				)
+			)
+		)
+	)
+	(symbol
+		(lib_id "Librairie_symbole:XT60-M")
+		(at 26.67 34.29 270)
+		(mirror x)
+		(unit 1)
+		(exclude_from_sim no)
+		(in_bom yes)
+		(on_board yes)
+		(dnp no)
+		(property "Reference" "J9"
+			(at 22.86 29.2099 90)
+			(effects
+				(font
+					(size 1.27 1.27)
+				)
+				(justify right)
+			)
+		)
+		(property "Value" "XT60-M"
+			(at 22.86 31.7499 90)
+			(effects
+				(font
+					(size 1.27 1.27)
+				)
+				(justify right)
+			)
+		)
+		(property "Footprint" "XT60-M:AMASS_XT60-M"
+			(at 26.67 34.29 0)
+			(effects
+				(font
+					(size 1.27 1.27)
+				)
+				(justify bottom)
+				(hide yes)
+			)
+		)
+		(property "Datasheet" ""
+			(at 26.67 34.29 0)
+			(effects
+				(font
+					(size 1.27 1.27)
+				)
+				(hide yes)
+			)
+		)
+		(property "Description" ""
+			(at 26.67 34.29 0)
+			(effects
+				(font
+					(size 1.27 1.27)
+				)
+				(hide yes)
+			)
+		)
+		(property "MF" "AMASS"
+			(at 26.67 34.29 0)
+			(effects
+				(font
+					(size 1.27 1.27)
+				)
+				(justify bottom)
+				(hide yes)
+			)
+		)
+		(property "MAXIMUM_PACKAGE_HEIGHT" "16.00 mm"
+			(at 26.67 34.29 0)
+			(effects
+				(font
+					(size 1.27 1.27)
+				)
+				(justify bottom)
+				(hide yes)
+			)
+		)
+		(property "Package" "Package"
+			(at 26.67 34.29 0)
+			(effects
+				(font
+					(size 1.27 1.27)
+				)
+				(justify bottom)
+				(hide yes)
+			)
+		)
+		(property "Price" "None"
+			(at 26.67 34.29 0)
+			(effects
+				(font
+					(size 1.27 1.27)
+				)
+				(justify bottom)
+				(hide yes)
+			)
+		)
+		(property "Check_prices" "https://www.snapeda.com/parts/XT60-M/AMASS/view-part/?ref=eda"
+			(at 26.67 34.29 0)
+			(effects
+				(font
+					(size 1.27 1.27)
+				)
+				(justify bottom)
+				(hide yes)
+			)
+		)
+		(property "STANDARD" "IPC 7351B"
+			(at 26.67 34.29 0)
+			(effects
+				(font
+					(size 1.27 1.27)
+				)
+				(justify bottom)
+				(hide yes)
+			)
+		)
+		(property "PARTREV" "V1.2"
+			(at 26.67 34.29 0)
+			(effects
+				(font
+					(size 1.27 1.27)
+				)
+				(justify bottom)
+				(hide yes)
+			)
+		)
+		(property "SnapEDA_Link" "https://www.snapeda.com/parts/XT60-M/AMASS/view-part/?ref=snap"
+			(at 26.67 34.29 0)
+			(effects
+				(font
+					(size 1.27 1.27)
+				)
+				(justify bottom)
+				(hide yes)
+			)
+		)
+		(property "MP" "XT60-M"
+			(at 26.67 34.29 0)
+			(effects
+				(font
+					(size 1.27 1.27)
+				)
+				(justify bottom)
+				(hide yes)
+			)
+		)
+		(property "Description_1" "Plug; DC supply; XT60; male; PIN: 2; for cable; soldered; 30A; 500V"
+			(at 26.67 34.29 0)
+			(effects
+				(font
+					(size 1.27 1.27)
+				)
+				(justify bottom)
+				(hide yes)
+			)
+		)
+		(property "Availability" "In Stock"
+			(at 26.67 34.29 0)
+			(effects
+				(font
+					(size 1.27 1.27)
+				)
+				(justify bottom)
+				(hide yes)
+			)
+		)
+		(property "MANUFACTURER" "AMASS"
+			(at 26.67 34.29 0)
+			(effects
+				(font
+					(size 1.27 1.27)
+				)
+				(justify bottom)
+				(hide yes)
+			)
+		)
+		(pin "2"
+		)
+		(pin "1"
+		)
+		(instances
+			(project ""
+				(path "/1781f24e-6d21-4940-8f28-5db05927caba"
+					(reference "J9")
+					(unit 1)
+				)

Commit message: mise à jour PCB
Parts:
- removed R_Pull_Up1: 1 k, Resistor_SMD:R_0805_2012Metric, symbol Device:R
- removed R_SCL1, R_SDA1: 4,7k, Resistor_SMD:R_0805_2012Metric, symbol Device:R
- removed Raspberry5: CM5108032, Connector_PinSocket_2.54mm:PinSocket_2x20_P2.54mm_Vertical, symbol Librairie_symbole:CM5108032
- added J10: RPI5_40pins, Connector_PinSocket_2.54mm:PinSocket_2x20_P2.54mm_Vertical, symbol Connector_Generic:Conn_02x20_Odd_Even
- added R_SCL2, R_SDA2: 4,7k, Resistor_SMD:R_0805_2012Metric, symbol Device:R
- J9: footprint XT60-M:AMASS_XT60-M -> Connector_AMASS:AMASS_XT60-F_1x02_P7.20mm_Vertical
- SW1: footprint Button_Switch_THT:SW_DIP_SPSTx01_Slide_6.7x4.1mm_W7.62mm_P2.54mm_LowProfile -> Button_Switch_THT:SW_Slide_SPDT_Straight_CK_OS102011MS2Q
Connections:
- net GND: now also SW1.3 (C), J10.14 (Pin_14), J10.20 (Pin_20), J10.25 (Pin_25), J10.30 (Pin_30), J10.34 (Pin_34), J10.39 (Pin_39), J10.6 (Pin_6), J10.9 (Pin_9); no longer SW1.2 (B)
- net SCL: now also J10.5 (Pin_5), R_SCL2.1
- net SDA: now also J10.3 (Pin_3), R_SDA2.2
- net at SW1.1 (A): now also F1.2, Régulateur_de_tension1.2 (VIN); no longer Régulateur_de_tension1.1 (ON/OFF_CONTROL)
- net +5V(INPUT) renamed 5V
- net 5V: now also J10.2 (Pin_2), J10.4 (Pin_4)
- net CM5_3.3V(OUTPUT) renamed 3.3V
- net 3.3V: now also J10.1 (Pin_1), J10.17 (Pin_17), R_SCL2.2, R_SDA2.1
- new net: Régulateur_de_tension1.1 (ON/OFF_CONTROL), SW1.2 (B)
Other:
- note added: "Check : pinout.xyz pour les connectiques"
- note added: "Connecteur_Raspberry_Pi_5"
- moved on the sheet: SW1
