File: carte_RPI5_KiCad/carte_rpi5_kicad.kicad_pcb (KiCad board)
At the start: 2 copper layers, 156.2 x 67.4 mm, 32 parts, among them J10 RPI5_40pins

Commit message: maj
Parts:
- moved BMI055 24.0 mm to (70.1, 64.5), turned to 90 degrees
Routing:
- net SDA: track 215.5 -> 196.5 mm
- net 3.3V: track 305.0 -> 288.8 mm
- net SCL: track 190.9 -> 175.5 mm
Other:
- outline, holes or cut-outs redrawn

Commit message: maj
Parts:
- removed the G*** at (61.8, 103.8)
