File: Carte_dock/carte_dock/carte_dock.kicad_sch (KiCad schematic)
At the start: 0 parts

Commit message: Add carte dock
Parts:
- added ConnecteurESP32-S3-WROOM: Conn_02x15_Odd_Even, symbol Connector_Generic:Conn_02x15_Odd_Even
Connections:
- new net 3.3V: ConnecteurESP32-S3-WROOM.30 (Pin_30)
- new net ADC0: ConnecteurESP32-S3-WROOM.3 (Pin_3)
- new net ADC14: ConnecteurESP32-S3-WROOM.25 (Pin_25)
- new net ADC15: ConnecteurESP32-S3-WROOM.23 (Pin_23)
- new net ADC16: ConnecteurESP32-S3-WROOM.21 (Pin_21)
- new net ADC17: ConnecteurESP32-S3-WROOM.19 (Pin_19)
- new net ADC18: ConnecteurESP32-S3-WROOM.15 (Pin_15)
- new net ADC19: ConnecteurESP32-S3-WROOM.17 (Pin_17)
- new net ADC3: ConnecteurESP32-S3-WROOM.5 (Pin_5)
- new net ADC4: ConnecteurESP32-S3-WROOM.11 (Pin_11)
- new net ADC5: ConnecteurESP32-S3-WROOM.13 (Pin_13)
- new net ADC6: ConnecteurESP32-S3-WROOM.7 (Pin_7)
- new net ADC7: ConnecteurESP32-S3-WROOM.9 (Pin_9)
- new net D15: ConnecteurESP32-S3-WROOM.26 (Pin_26)
- new net D18: ConnecteurESP32-S3-WROOM.14 (Pin_14)
- new net D19: ConnecteurESP32-S3-WROOM.12 (Pin_12)
- new net D2: ConnecteurESP32-S3-WROOM.24 (Pin_24)
- new net D21: ConnecteurESP32-S3-WROOM.10 (Pin_10)
- new net D22: ConnecteurESP32-S3-WROOM.4 (Pin_4)
- new net D23: ConnecteurESP32-S3-WROOM.2 (Pin_2)
- new net D4: ConnecteurESP32-S3-WROOM.22 (Pin_22)
- new net D5: ConnecteurESP32-S3-WROOM.16 (Pin_16)
- new net EN: ConnecteurESP32-S3-WROOM.1 (Pin_1)
- new net GND: ConnecteurESP32-S3-WROOM.27 (Pin_27), ConnecteurESP32-S3-WROOM.28 (Pin_28)
- new net RX0: ConnecteurESP32-S3-WROOM.8 (Pin_8)
- new net RX2: ConnecteurESP32-S3-WROOM.20 (Pin_20)
- new net TX0: ConnecteurESP32-S3-WROOM.6 (Pin_6)
- new net TX2: ConnecteurESP32-S3-WROOM.18 (Pin_18)
- new net Vin: ConnecteurESP32-S3-WROOM.29 (Pin_29)
