File: carte_dock_elec/carte_elec_Kicad/carte_dock_elec_kicad/carte_dock_elec_kicad.kicad_pcb (KiCad board)
At the start: 2 copper layers, 13 parts, among them J1 1758018, J10 Conn_02x20_Odd_Even, J2 22053021, J3 22272041, J4 22272041, J5 22272041, J6 1758018, J7 1758018, J8 1758018, J9 1758018, Q1 IRLB8748PBF

Commit message: carte_dock
Parts:
- moved D1 103.0 mm to (101.8, 75.0)
- moved Q1 100.6 mm to (82.5, 78.4), turned to -90 degrees
- moved J8 95.9 mm to (103.7, 69.0)
- moved R1 92.9 mm to (101.3, 89.5)
- moved J6 89.9 mm to (85.0, 57.0), turned to 180 degrees
- moved J7 87.1 mm to (90.0, 69.0)
- moved J1 76.7 mm to (103.5, 57.5)
- moved J9 76.3 mm to (95.5, 99.5), turned to -90 degrees
- moved J2 75.9 mm to (99.4, 82.0), turned to 90 degrees
- moved J5 73.9 mm to (75.0, 91.8), turned to 90 degrees
- moved J4 64.3 mm to (90.9, 84.6), turned to -90 degrees
- moved J3 55.2 mm to (83.0, 91.9), turned to 90 degrees
- moved J10 52.1 mm to (66.5, 99.7), turned to 180 degrees
Connections:
- J10 pad 1: 3.3V -> 5V
- J10 pad 11: PIN11 -> unconnected-(J10-Pin_11-Pad11)
- J10 pad 12: unconnected-(J10-Pin_12-Pad12) -> PIN11
- J10 pad 13: PIN13 -> unconnected-(J10-Pin_13-Pad13)
- J10 pad 14: unconnected-(J10-Pin_14-Pad14) -> PIN13
- J10 pad 15: PIN15 -> unconnected-(J10-Pin_15-Pad15)
- J10 pad 16: unconnected-(J10-Pin_16-Pad16) -> PIN15
- J10 pad 2: 5V -> 3.3V
- J10 pad 3: SDA -> 5V
- J10 pad 4: 5V -> SDA
- J10 pad 5: SCL -> unconnected-(J10-Pin_5-Pad5)
- J10 pad 6: unconnected-(J10-Pin_6-Pad6) -> SCL
Routing:
- net GND: track 0.00 -> 85.5 mm
- net 5V: track 0.00 -> 66.8 mm
- net Net-(D1-K): track 0.00 -> 46.8 mm
- net PIN13: track 0.00 -> 39.4 mm
- net Net-(D1-A): track 0.00 -> 36.5 mm
- net PIN11: track 0.00 -> 22.8 mm
- net PIN15: track 0.00 -> 14.9 mm
- net SDA: track 0.00 -> 14.1 mm
- net SCL: track 0.00 -> 14.1 mm
- net 3.3V: track 0.00 -> 14.1 mm

Commit message: carte_dock_helium
Routing:
- net 5V: track 66.8 -> 69.4 mm
- net GND: track 85.5 -> 84.8 mm
- added copper zone on B.Cu, net GND
- added copper zone on F.Cu, net GND

Commit message: MAJ DOCK ELEC
Parts:
- D1: footprint Diode_SMD:D_0201_0603Metric -> Diode_SMD:D_1206_3216Metric
- R1: footprint Resistor_SMD:R_0201_0603Metric -> Resistor_SMD:R_1206_3216Metric
Routing:
- net GND: track 84.8 -> 23.1 mm
- net PIN13: track 39.4 -> 51.7 mm
- net Net-(D1-A): track 36.5 -> 37.6 mm
Other:
- board outline added: 50.5 x 57.9 mm

Commit message: modif PCB_carte_doc
Parts:
- D1, R1: moved to B.Cu
- moved R1 0.63 mm to (101.0, 90.0)
Routing:
- net PIN13: track 51.7 -> 9.78 mm
- net Net-(D1-K): track 46.6 -> 34.1 mm
- net 5V: track 69.0 -> 71.2 mm
- net Net-(D1-A): track 37.6 -> 38.5 mm

Commit message: rapport
Parts:
- added J11: 1758018, Librarie_empreinte:CONN_1758018, F.Cu at (79.0, 58.5)
- added J12: 1758018, Librarie_empreinte:CONN_1758018, F.Cu at (79.0, 68.8)
Connections:
- J10 pad 15: unconnected-(J10-Pin_15-Pad15) -> PIN16
- J10 pad 30: unconnected-(J10-Pin_30-Pad30) -> PIN29
Routing:
- net PIN16: track 0.00 -> 49.4 mm
- net PIN13: track 9.78 -> 48.9 mm, vias 0 -> 2
- net Net-(D1-K): track 34.1 -> 67.1 mm
- net GND: track 23.1 -> 1.35 mm
- net PIN29: track 0.00 -> 13.2 mm
- net Net-(D1-A): track 38.5 -> 40.7 mm

Commit message: modif_carte_dick
Connections:
- J10 pad 5: unconnected-(J10-Pin_5-Pad5) -> GND
Routing:
- net PIN13: track 48.9 -> 44.8 mm
Other:
- board text added: "Bot"
- board text added: "Front"
Changed lines of the file:
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@@
 			(layers "*.Cu" "*.Mask")
 			(remove_unused_layers no)
-			(net "unconnected-(J10-Pin_5-Pad5)")
+			(net "GND")
 			(pinfunction "Pin_5_5")
 			(pintype "passive")
@@
 		(layer "Edge.Cuts")
 	)
+	(gr_text "Front\n"
+		(at 105 95.5 0)
+		(layer "F.Cu" knockout)
+		(effects
+			(font
+				(size 1.5 1.5)
+				(thickness 0.3)
+				(bold yes)
+			)
+			(justify left bottom)
+		)
+	)
+	(gr_text "Bot\n"
+		(at 110.5 93 0)
+		(layer "B.Cu" knockout)
+		(effects
+			(font
+				(size 1.5 1.5)
+				(thickness 0.3)
+				(bold yes)
+			)
+			(justify left bottom mirror)
+		)
+	)
 	(segment
 		(start 82.96 91.84)
@@
 	)
 	(segment
+		(start 73.937 58.530216)
+		(end 73.937 53.063)
+		(width 0.5)
+		(layer "B.Cu")
+		(net "PIN16")
+	)
+	(segment
+		(start 64.5 50)
+		(end 64.5 79.96)
+		(width 0.5)
+		(layer "B.Cu")
+		(net "PIN16")
+	)
+	(segment
+		(start 64.5 79.96)
+		(end 66.46 81.92)
+		(width 0.5)
+		(layer "B.Cu")
+		(net "PIN16")
+	)
+	(segment
+		(start 74 53)
+		(end 70.5 49.5)
+		(width 0.5)
+		(layer "B.Cu")
+		(net "PIN16")
+	)
+	(segment
+		(start 70.5 49.5)
+		(end 65 49.5)
+		(width 0.5)
+		(layer "B.Cu")
+		(net "PIN16")
+	)
+	(segment
+		(start 73.937 53.063)
+		(end 74 53)
+		(width 0.5)
+		(layer "B.Cu")
+		(net "PIN16")
+	)
+	(segment
+		(start 65 49.5)
+		(end 64.5 50)
+		(width 0.5)
+		(layer "B.Cu")
+		(net "PIN16")
+	)
+	(segment
+		(start 74.827216 64.14)
+		(end 69 64.14)
+		(width 0.5)
+		(layer "B.Cu")
+		(net "PIN29")
+	)
+	(segment
+		(start 79 59.967216)
+		(end 74.827216 64.14)
+		(width 0.5)
+		(layer "B.Cu")
+		(net "PIN29")
+	)
+	(segment
+		(start 79 58.5)
+		(end 79 59.967216)
+		(width 0.5)
+		(layer "B.Cu")
+		(net "PIN29")
+	)
+	(segment
 		(start 103.5 57.5)
 		(end 103.5 64.11)
@@
 	)
 	(segment
-		(start 89.5 88.5)
-		(end 80.5 88.5)
+		(start 76.5 84.5)
+		(end 74.5 84.5)
+		(width 0.5)
+		(layer "F.Cu")
+		(net "PIN13")
+	)
+	(segment
+		(start 99.4294 84.7211)
+		(end 99.4294 87.0706)
 		(width 0.5)
 		(layer "F.Cu")
@@
 	)
 	(segment
-		(start 102 84.5)
+		(start 99.4294 87.0706)
 		(end 98 88.5)
 		(width 0.5)
@@
 	(segment
 		(start 98 88.5)
-		(end 89.5 88.5)
+		(end 80.5 88.5)
 		(width 0.5)
 		(layer "F.Cu")
@@
 	)
 	(segment
-		(start 76.5 84.5)
-		(end 74.5 84.5)
+		(start 80.5 88.5)
+		(end 76.5 84.5)
 		(width 0.5)
 		(layer "F.Cu")
@@
 		(net "PIN13")
 	)
-	(segment
-		(start 80.5 88.5)
-		(end 76.5 84.5)
-		(width 0.5)
-		(layer "F.Cu")
-		(net "PIN13")
-	)
 	(via
 		(at 74.5 84.5)
-		(size 1)
-		(drill 0.7)
+		(size 1.5)
+		(drill 0.8)
 		(layers "F.Cu" "B.Cu")
-		(locked yes)
 		(free yes)
 		(net "PIN13")
 	)
 	(via
-		(at 102 84.5)
-		(size 1)
-		(drill 0.7)
+		(at 99.4294 84.7211)
+		(size 1.5)
+		(drill 0.8)
 		(layers "F.Cu" "B.Cu")
-		(locked yes)
 		(free yes)
 		(net "PIN13")
@@
 	)
 	(segment
-		(start 99.60415 84.89585)
-		(end 101.60415 84.89585)
-		(width 0.5)
-		(layer "B.Cu")
-		(net "PIN13")
-	)
-	(segment
 		(start 69.04 84.5)
 		(end 69 84.46)
@@
 	(segment
 		(start 99.4294 84.7211)
-		(end 99.60415 84.89585)
-		(width 1)
-		(layer "B.Cu")
-		(net "PIN13")
-	)
-	(segment
-		(start 101.60415 84.89585)
-		(end 102 84.5)
-		(width 1)
-		(layer "B.Cu")
-		(net "PIN13")
-	)
-	(segment
-		(start 99.4294 84.7211)
 		(end 99.4294 82.0381)
 		(width 0.5)
@@
 		(net "Net-(D1-A)")
 	)
-	(segment
-		(start 73.937 58.530216)
-		(end 73.937 53.063)
-		(width 0.5)
-		(layer "B.Cu")
-		(net "PIN16")
-	)
-	(segment
-		(start 64.5 50)
-		(end 64.5 79.96)
-		(width 0.5)
-		(layer "B.Cu")
-		(net "PIN16")
-	)
-	(segment
-		(start 64.5 79.96)
-		(end 66.46 81.92)
-		(width 0.5)
-		(layer "B.Cu")
-		(net "PIN16")
-	)
-	(segment
-		(start 74 53)
-		(end 70.5 49.5)
-		(width 0.5)
-		(layer "B.Cu")
-		(net "PIN16")
-	)
-	(segment
-		(start 70.5 49.5)
-		(end 65 49.5)
-		(width 0.5)
-		(layer "B.Cu")
-		(net "PIN16")
-	)
-	(segment
-		(start 73.937 53.063)
-		(end 74 53)
-		(width 0.5)
-		(layer "B.Cu")
-		(net "PIN16")
-	)
-	(segment
-		(start 65 49.5)
-		(end 64.5 50)
-		(width 0.5)
-		(layer "B.Cu")
-		(net "PIN16")
-	)
-	(segment
-		(start 74.827216 64.14)
-		(end 69 64.14)
-		(width 0.5)
-		(layer "B.Cu")
-		(net "PIN29")
-	)
-	(segment
-		(start 79 59.967216)
-		(end 74.827216 64.14)
-		(width 0.5)
-		(layer "B.Cu")
-		(net "PIN29")
-	)
-	(segment
-		(start 79 58.5)
-		(end 79 59.967216)
-		(width 0.5)
-		(layer "B.Cu")
-		(net "PIN29")
-	)
 	(zone
